File: kicad files/led_web.kicad_sch (KiCad schematic)
At the start: 5 parts, among them U1 MAX4466, U2 WeMos_D1_mini, U3 SSD1306

Commit message: pcb redesign
Parts:
- added RV1: R_Potentiometer, Potentiometer_THT:Potentiometer_Runtron_RM-065_Vertical, symbol Device:R_Potentiometer
- U1: value MAX4466 -> SSD1306; footprint led_web_foots:MAX4466 -> led_web_foots:SSD1306
- U3: value SSD1306 -> (none); footprint led_web_foots:SSD1306 -> (none)
Connections:
- net GND: now also U1.4 (GND); no longer U1.2 (GND)
- net at U2.13 (SDA/D2): now also U1.1 (SDA); no longer U1.4 (SDA)
- net at U2.14 (SCL/D1): now also U1.2 (SCL); no longer U1.3 (SCL)
- net at U2.2 (A0): now also RV1.2; no longer U3.3 (OUT)
- net at C1.1, L1.1 (VCC), U2.9 (5V): now also U1.3 (VCC), U3.3 (VCC); no longer U1.1 (VCC), U3.1 (VCC)
- new net: RV1.1, U3.1 (OUT)
Other:
- moved on the sheet: U1
Changed lines of the file:
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@@
   (title_block
     (title "LED_WEB")
-    (date "2022-03-14")
-    (rev "V1")
+    (date "2022-08-02")
+    (rev "V2")
     (comment 1 "NOT TO BE COPIED WITHOUT PERMISSION")
   )
@@
     (stroke (width 0) (type default) (color 0 0 0 0))
   )
-  (wire (pts (xy 125.73 116.84) (xy 120.65 116.84))
+  (wire (pts (xy 125.73 116.84) (xy 123.19 116.84))
     (stroke (width 0) (type default) (color 255 0 0 1))
   )
@@
     (stroke (width 0) (type default) (color 0 0 0 1))
   )
-  (wire (pts (xy 109.22 99.06) (xy 140.97 99.06))
-    (stroke (width 0) (type default) (color 0 0 0 0))
-  )
-  (wire (pts (xy 120.65 92.71) (xy 129.54 92.71))
+  (wire (pts (xy 120.65 99.06) (xy 140.97 99.06))
+    (stroke (width 0) (type default) (color 0 0 0 0))
+  )
+  (wire (pts (xy 113.03 92.71) (xy 129.54 92.71))
     (stroke (width 0) (type default) (color 255 0 0 1))
   )
@@
     (stroke (width 0) (type default) (color 0 0 0 1))
   )
-  (wire (pts (xy 173.99 81.28) (xy 173.99 85.09))
+  (wire (pts (xy 168.91 85.09) (xy 168.91 81.28))
     (stroke (width 0) (type default) (color 255 0 0 1))
   )
@@
     (stroke (width 0) (type default) (color 255 0 0 1))
   )
-  (wire (pts (xy 133.35 82.55) (xy 133.35 104.14))
-    (stroke (width 0) (type default) (color 0 0 0 0))
-  )
-  (wire (pts (xy 120.65 116.84) (xy 120.65 97.79))
+  (wire (pts (xy 113.03 81.28) (xy 113.03 80.01))
+    (stroke (width 0) (type default) (color 0 0 0 0))
+  )
+  (wire (pts (xy 133.35 78.74) (xy 133.35 104.14))
+    (stroke (width 0) (type default) (color 0 0 0 0))
+  )
+  (wire (pts (xy 123.19 116.84) (xy 123.19 97.79))
     (stroke (width 0) (type solid) (color 255 0 0 1))
   )
@@
     (stroke (width 0) (type default) (color 0 0 0 1))
   )
+  (wire (pts (xy 173.99 82.55) (xy 173.99 81.28))
+    (stroke (width 0) (type default) (color 0 0 0 0))
+  )
   (wire (pts (xy 171.45 81.28) (xy 171.45 88.9))
     (stroke (width 0) (type default) (color 0 0 0 1))
@@
     (stroke (width 0) (type default) (color 0 0 0 1))
   )
-  (wire (pts (xy 120.65 97.79) (xy 140.97 97.79))
-    (stroke (width 0) (type default) (color 255 0 0 1))
-  )
-  (wire (pts (xy 116.84 81.28) (xy 116.84 86.36))
-    (stroke (width 0) (type default) (color 0 0 0 1))
-  )
-  (wire (pts (xy 113.03 101.6) (xy 138.43 101.6))
-    (stroke (width 0) (type default) (color 0 0 0 0))
-  )
-  (wire (pts (xy 113.03 81.28) (xy 113.03 101.6))
-    (stroke (width 0) (type default) (color 0 0 0 0))
-  )
-  (wire (pts (xy 109.22 81.28) (xy 109.22 99.06))
+  (wire (pts (xy 123.19 97.79) (xy 140.97 97.79))
+    (stroke (width 0) (type default) (color 255 0 0 1))
+  )
+  (wire (pts (xy 109.22 80.01) (xy 109.22 85.09))
+    (stroke (width 0) (type default) (color 0 0 0 1))
+  )
+  (wire (pts (xy 116.84 101.6) (xy 138.43 101.6))
+    (stroke (width 0) (type default) (color 0 0 0 0))
+  )
+  (wire (pts (xy 116.84 80.01) (xy 116.84 101.6))
+    (stroke (width 0) (type default) (color 0 0 0 0))
+  )
+  (wire (pts (xy 120.65 80.01) (xy 120.65 99.06))
     (stroke (width 0) (type default) (color 0 0 0 0))
   )
@@
     (stroke (width 0) (type default) (color 255 0 0 1))
   )
-  (wire (pts (xy 135.89 85.09) (xy 173.99 85.09))
+  (wire (pts (xy 135.89 85.09) (xy 168.91 85.09))
     (stroke (width 0) (type default) (color 255 0 0 1))
   )
@@
     (stroke (width 0) (type default) (color 255 0 0 1))
   )
-  (wire (pts (xy 168.91 81.28) (xy 168.91 82.55))
-    (stroke (width 0) (type default) (color 0 0 0 0))
-  )
-  (wire (pts (xy 120.65 81.28) (xy 120.65 92.71))
-    (stroke (width 0) (type default) (color 255 0 0 1))
-  )
-  (wire (pts (xy 168.91 82.55) (xy 133.35 82.55))
-    (stroke (width 0) (type default) (color 0 0 0 0))
+  (wire (pts (xy 113.03 81.28) (xy 113.03 92.71))
+    (stroke (width 0) (type default) (color 255 0 0 1))
   )
   (wire (pts (xy 96.52 93.98) (xy 96.52 129.54))
+    (stroke (width 0) (type default) (color 0 0 0 0))
+  )
+  (wire (pts (xy 154.94 82.55) (xy 173.99 82.55))
+    (stroke (width 0) (type default) (color 0 0 0 0))
+  )
+  (wire (pts (xy 133.35 78.74) (xy 151.13 78.74))
     (stroke (width 0) (type default) (color 0 0 0 0))
   )
@@
     (pin "1")
   )
-  (symbol (lib_id "power:GND") (at 116.84 86.36 0) (unit 1)
-    (in_bom yes) (on_board yes) (fields_autoplaced)
-    (property "Reference" "#PWR02" (id 0) (at 116.84 92.71 0)
-      (effects (font (size 1.27 1.27)) hide)
-    )
-    (property "Value" "GND" (id 1) (at 116.84 91.44 0))
-    (property "Footprint" "" (id 2) (at 116.84 86.36 0)
-      (effects (font (size 1.27 1.27)) hide)
-    )
-    (property "Datasheet" "" (id 3) (at 116.84 86.36 0)
+  (symbol (lib_id "power:GND") (at 109.22 85.09 0) (unit 1)
+    (in_bom yes) (on_board yes)
+    (property "Reference" "#PWR02" (id 0) (at 109.22 91.44 0)
+      (effects (font (size 1.27 1.27)) hide)
+    )
+    (property "Value" "GND" (id 1) (at 106.68 85.09 0))
+    (property "Footprint" "" (id 2) (at 109.22 85.09 0)
+      (effects (font (size 1.27 1.27)) hide)
+    )
+    (property "Datasheet" "" (id 3) (at 109.22 85.09 0)
       (effects (font (size 1.27 1.27)) hide)
     )
@@
     (pin "3")
   )
-  (symbol (lib_id "led_web_sym:SSD1306") (at 114.935 76.2 0) (unit 1)
-    (in_bom yes) (on_board yes)
-    (property "Reference" "U1" (id 0) (at 106.68 72.39 0)
-      (effects (font (size 1.27 1.27)) (justify left))
-    )
-    (property "Value" "MAX4466" (id 1) (at 123.825 78.7399 0)
-      (effects (font (size 1.27 1.27)) (justify left))
-    )
-    (property "Footprint" "led_web_foots:MAX4466" (id 2) (at 113.665 73.66 0)
-      (effects (font (size 1.27 1.27)) hide)
-    )
-    (property "Datasheet" "" (id 3) (at 113.665 73.66 0)
+  (symbol (lib_id "led_web_sym:SSD1306") (at 114.3 74.93 0) (unit 1)
+    (in_bom yes) (on_board yes)
+    (property "Reference" "U1" (id 0) (at 106.045 71.12 0)
+      (effects (font (size 1.27 1.27)) (justify left))
+    )
+    (property "Value" "SSD1306" (id 1) (at 123.19 77.4699 0)
+      (effects (font (size 1.27 1.27)) (justify left))
+    )
+    (property "Footprint" "led_web_foots:SSD1306" (id 2) (at 113.03 72.39 0)
+      (effects (font (size 1.27 1.27)) hide)
+    )
+    (property "Datasheet" "" (id 3) (at 113.03 72.39 0)
       (effects (font (size 1.27 1.27)) hide)
     )
@@
     (pin "1")
   )
+  (symbol (lib_id "Device:R_Potentiometer") (at 151.13 82.55 270) (mirror x) (unit 1)
+    (in_bom yes) (on_board yes)
+    (property "Reference" "RV1" (id 0) (at 154.94 78.74 90))
+    (property "Value" "R_Potentiometer" (id 1) (at 149.86 76.2 90))
+    (property "Footprint" "Potentiometer_THT:Potentiometer_Runtron_RM-065_Vertical" (id 2) (at 151.13 82.55 0)
+      (effects (font (size 1.27 1.27)) hide)
+    )
+    (property "Datasheet" "~" (id 3) (at 151.13 82.55 0)
+      (effects (font (size 1.27 1.27)) hide)
+    )
+    (pin "1")
+    (pin "2")
+    (pin "3")
+  )
   (symbol (lib_id "led_web_sym:MAX4466") (at 171.45 83.185 0) (unit 1)
     (in_bom yes) (on_board yes)
@@
       (effects (font (size 1.27 1.27)) (justify left))
     )
-    (property "Value" "SSD1306" (id 1) (at 176.53 77.7874 0)
-      (effects (font (size 1.27 1.27)) (justify left))
-    )
-    (property "Footprint" "led_web_foots:SSD1306" (id 2) (at 171.45 83.185 0)
+    (property "Value" "" (id 1) (at 176.53 77.7874 0)
+      (effects (font (size 1.27 1.27)) (justify left))
+    )
+    (property "Footprint" "" (id 2) (at 171.45 83.185 0)
       (effects (font (size 1.27 1.27)) hide)
     )
@@
       (reference "L1") (unit 1) (value "LED_STRIP") (footprint "led_web_foots:LED_STRIP")
     )
+    (path "/be679199-4dd7-4cff-ba3d-8a47068afa40"
+      (reference "RV1") (unit 1) (value "R_Potentiometer") (footprint "Potentiometer_THT:Potentiometer_Runtron_RM-065_Vertical")
+    )
     (path "/a9e8bc25-1779-42c1-9b3a-ae61e8b0700f"
-      (reference "U1") (unit 1) (value "MAX4466") (footprint "led_web_foots:MAX4466")
+      (reference "U1") (unit 1) (value "SSD1306") (footprint "led_web_foots:SSD1306")
     )
     (path "/0f262423-d4d1-4f04-805d-93d3f5b41978"
@@
     )
     (path "/f1b5c05a-d227-4ea7-9d1f-3663511dd723"
-      (reference "U3") (unit 1) (value "SSD1306") (footprint "led_web_foots:SSD1306")
-    )
-  )
+      (reference "U3") (unit 1) (value "MAX4466") (footprint "led_web_foots:MAX4466")
+    )
+  )
